Commit message: Add imu and lidar gazebo bringup

File: src/maya_description/urdf/maya_description.urdf.xacro (robot description, xacro)
@@ -1,4 +1,5 @@
 <?xml version="1.0"?>
-<robot name="maya" xmlns:xacro="http://www.ros.org/wiki/xacro">
+<robot name="maya"
+  xmlns:xacro="http://www.ros.org/wiki/xacro">
   <!-- brief Top level robot description for Maya Rover -->
   <!-- This file aggregates shared properties, physical model and Gazebo plugins -->
@@ -6,3 +7,4 @@
   <xacro:include filename="$(find maya_description)/urdf/mobile_base.xacro"/>
   <xacro:include filename="$(find maya_description)/urdf/mobile_base_gazebo.xacro"/>
+  <xacro:include filename="$(find maya_description)/urdf/sensors.xacro"/>
 </robot>

File: src/maya_description/urdf/mobile_base.xacro (robot description, xacro)
@@ -4,16 +4,9 @@
   <link name="base_link">
     <!-- Base inertia approximated as axis-aligned box using base dimensions -->
-    <xacro:box_inertia
-      m="${base_mass}"
-      w="${base_width}"
-      d="${base_length}"
-      h="${base_height}"
-      xyz="${base_inertial_xyz}"
-      rpy="${base_inertial_rpy}"/>
+    <xacro:box_inertia m="${base_mass}" w="${base_width}" d="${base_length}" h="${base_height}" xyz="${base_inertial_xyz}" rpy="${base_inertial_rpy}"/>
     <visual>
       <origin xyz="${base_link_mesh_offset_xyz}" rpy="${base_link_mesh_offset_rpy}"/>
       <geometry>
-        <mesh filename="file://$(find maya_description)/meshes/base_link.STL"
-              scale="${mesh_scale} ${mesh_scale} ${mesh_scale}"/>
+        <mesh filename="file://$(find maya_description)/meshes/base_link.STL" scale="${mesh_scale} ${mesh_scale} ${mesh_scale}"/>
       </geometry>
       <material name="maya_body"/>
@@ -22,6 +15,5 @@
       <origin xyz="${base_link_mesh_offset_xyz}" rpy="${base_link_mesh_offset_rpy}"/>
       <geometry>
-        <mesh filename="file://$(find maya_description)/meshes/base_link.STL"
-              scale="${mesh_scale} ${mesh_scale} ${mesh_scale}"/>
+        <mesh filename="file://$(find maya_description)/meshes/base_link.STL" scale="${mesh_scale} ${mesh_scale} ${mesh_scale}"/>
       </geometry>
     </collision>
@@ -32,27 +24,18 @@
   <joint name="base_joint" type="fixed">
     <parent link="base_footprint"/>
-    <child  link="base_link"/>
+    <child link="base_link"/>
     <!-- Rotate robot body so that physical forward aligns with base_footprint X -->
     <origin xyz="0 0 ${footprint_z}" rpy="0 0 ${half_pi}"/>
   </joint>
   <!-- Generic wheel macro with inertial, visual and continuous joint -->
-  <xacro:macro name="maya_wheel"
-               params="prefix mesh
-                       xyz:='0 0 0' rpy:='0 0 0' axis:='${wheel_axis_left}'
-                       inertial_xyz:='0 0 0' inertial_rpy:='0 0 0'">
+  <xacro:macro name="maya_wheel" params="prefix mesh xyz:='0 0 0' rpy:='0 0 0' axis:='${wheel_axis_left}' inertial_xyz:='0 0 0' inertial_rpy:='0 0 0'">
     <link name="${prefix}">
       <!-- Wheel inertia approximated as solid cylinder
            COM and orientation taken from inertial_xyz / inertial_rpy -->
-      <xacro:cylinder_inertia
-        m="${wheel_mass}"
-        r="${wheel_radius}"
-        h="${wheel_width}"
-        xyz="${inertial_xyz}"
-        rpy="${inertial_rpy}"/>
+      <xacro:cylinder_inertia m="${wheel_mass}" r="${wheel_radius}" h="${wheel_width}" xyz="${inertial_xyz}" rpy="${inertial_rpy}"/>
       <visual>
         <origin xyz="0 0 0" rpy="0 0 0"/>
         <geometry>
-          <mesh filename="${mesh}"
-                scale="${mesh_scale} ${mesh_scale} ${mesh_scale}"/>
+          <mesh filename="${mesh}" scale="${mesh_scale} ${mesh_scale} ${mesh_scale}"/>
         </geometry>
         <material name="maya_wheel"/>
@@ -61,6 +44,5 @@
         <origin xyz="0 0 0" rpy="0 0 0"/>
         <geometry>
-          <mesh filename="${mesh}"
-                scale="${mesh_scale} ${mesh_scale} ${mesh_scale}"/>
+          <mesh filename="${mesh}" scale="${mesh_scale} ${mesh_scale} ${mesh_scale}"/>
         </geometry>
       </collision>
@@ -68,5 +50,5 @@
     <joint name="${prefix}_joint" type="continuous">
       <parent link="base_link"/>
-      <child  link="${prefix}"/>
+      <child link="${prefix}"/>
       <origin xyz="${xyz}" rpy="${rpy}"/>
       <axis xyz="${axis}"/>
@@ -74,34 +56,8 @@
   </xacro:macro>
   <!-- Left wheels use default spin axis from wheel_axis_left -->
-  <xacro:maya_wheel
-      prefix="front_left"
-      mesh="file://$(find maya_description)/meshes/front_left.STL"
-      xyz="-0.38478 -0.62736 -0.27744"
-      rpy="1.5702 0 1.5708"
-      inertial_xyz="-4.8481E-06 -8.0801E-06 -0.057753"
-      inertial_rpy="0 0 0"/>
-  <xacro:maya_wheel
-      prefix="back_left"
-      mesh="file://$(find maya_description)/meshes/back_left.STL"
-      xyz="-0.38513 0.28848 -0.27699"
-      rpy="1.5708 0 1.5708"
-      inertial_xyz="-4.8481E-06 -8.0801E-06 -0.057572"
-      inertial_rpy="0 0 0"/>
+  <xacro:maya_wheel prefix="front_left" mesh="file://$(find maya_description)/meshes/front_left.STL" xyz="-0.38478 -0.62736 -0.27744" rpy="1.5702 0 1.5708" inertial_xyz="-4.8481E-06 -8.0801E-06 -0.057753" inertial_rpy="0 0 0"/>
+  <xacro:maya_wheel prefix="back_left" mesh="file://$(find maya_description)/meshes/back_left.STL" xyz="-0.38513 0.28848 -0.27699" rpy="1.5708 0 1.5708" inertial_xyz="-4.8481E-06 -8.0801E-06 -0.057572" inertial_rpy="0 0 0"/>
   <!-- Right wheels override spin axis to wheel_axis_right -->
-  <xacro:maya_wheel
-      prefix="front_right"
-      mesh="file://$(find maya_description)/meshes/front_right.STL"
-      xyz="0.3987596 -0.61714 -0.27409"
-      rpy="1.5657 0.51887 -1.5734"
-      axis="${wheel_axis_right}"
-      inertial_xyz="-4.8512E-06 -8.0627E-06 -0.046342"
-      inertial_rpy="0 0 0"/>
-  <xacro:maya_wheel
-      prefix="back_right"
-      mesh="file://$(find maya_description)/meshes/back_right.STL"
-      xyz="0.4012382 0.27364 -0.28031"
-      rpy="-1.5781 -0.91737 1.5766"
-      axis="${wheel_axis_right}"
-      inertial_xyz="-4.8659E-06 -8.069E-06 -0.034709"
-      inertial_rpy="0 0 0"/>
+  <xacro:maya_wheel prefix="front_right" mesh="file://$(find maya_description)/meshes/front_right.STL" xyz="0.3987596 -0.61714 -0.27409" rpy="1.5657 0.51887 -1.5734" axis="${wheel_axis_right}" inertial_xyz="-4.8512E-06 -8.0627E-06 -0.046342" inertial_rpy="0 0 0"/>
+  <xacro:maya_wheel prefix="back_right" mesh="file://$(find maya_description)/meshes/back_right.STL" xyz="0.4012382 0.27364 -0.28031" rpy="-1.5781 -0.91737 1.5766" axis="${wheel_axis_right}" inertial_xyz="-4.8659E-06 -8.069E-06 -0.034709" inertial_rpy="0 0 0"/>
 </robot>

File: src/maya_description/urdf/mobile_base_gazebo.xacro (robot description, xacro)
@@ -19,6 +19,12 @@
   </gazebo>
   <gazebo>
-    <plugin filename="gz-sim-joint-state-publisher-system"
-            name="gz::sim::systems::JointStatePublisher">
+    <plugin filename="gz-sim-joint-state-publisher-system" name="gz::sim::systems::JointStatePublisher">
+    </plugin>
+  </gazebo>
+  <gazebo>
+    <plugin filename="gz-sim-imu-system" name="gz::sim::systems::Imu">
+    </plugin>
+    <plugin filename="gz-sim-sensors-system" name="gz::sim::systems::Sensors">
+      <render_engine>ogre2</render_engine>
     </plugin>
   </gazebo>
