Commit message: Checkpoint GNSS global navigation scaffold
Document the parked Nav2 GPS/global-localization branch and the direct GNSS waypoint architecture plan.\n\nKeep stable sim defaults on random_world with GPS localization disabled, while preserving explicit GPS/Nav2 experiment wiring, Gazebo NavSat scaffolding, GNSS covariance relay, and georeferenced worlds.

File: src/maya_description/urdf/sensors_frames.xacro (robot description, xacro)
@@ -13,4 +13,19 @@
     <child link="imu_link"/>
     <origin xyz="0 0 0" rpy="0 0 0"/>
+  </joint>
+  <!-- GNSS Link and Joint.
+       Keep this frame/topic naming aligned with Kukulcan firmware.
+       /sensors/gnss/fix stamped in frame gnss_link. -->
+  <link name="gnss_link">
+    <inertial>
+      <mass value="0.01"/>
+      <origin xyz="0 0 0" rpy="0 0 0"/>
+      <inertia ixx="0.00001" ixy="0" ixz="0" iyy="0.00001" iyz="0" izz="0.00001"/>
+    </inertial>
+  </link>
+  <joint name="gnss_joint" type="fixed">
+    <parent link="base_link"/>
+    <child link="gnss_link"/>
+    <origin xyz="0 0 0.20" rpy="0 0 0"/>
   </joint>
   <!-- LiDAR Link and Joint -->

File: src/maya_description/urdf/sensors_gazebo.xacro (robot description, xacro)
@@ -55,4 +55,34 @@
         </linear_acceleration>
       </imu>
+    </sensor>
+  </gazebo>
+  <!-- GNSS/NavSat Sensor Plugin
+       Sim publishes the same topic/frame as Kukulcan firmware so downstream
+       localization does not care whether sim or hardware is the source. -->
+  <gazebo reference="gnss_link">
+    <sensor name="gnss_sensor" type="navsat">
+      <always_on>true</always_on>
+      <update_rate>5</update_rate>
+      <visualize>true</visualize>
+      <topic>/sensors/gnss/fix</topic>
+      <gz_frame_id>gnss_link</gz_frame_id>
+      <navsat>
+        <position_sensing>
+          <horizontal>
+            <noise type="gaussian">
+              <mean>0.0</mean>
+              <!-- Gazebo NavSat horizontal noise is applied in geographic coordinates;
+                   keep sim noise at zero here and model GPS trust via ROS covariance. -->
+              <stddev>0.0</stddev>
+            </noise>
+          </horizontal>
+          <vertical>
+            <noise type="gaussian">
+              <mean>0.0</mean>
+              <stddev>0.0</stddev>
+            </noise>
+          </vertical>
+        </position_sensing>
+      </navsat>
     </sensor>
   </gazebo>
