Commit message: Fix base and wheel inertial properties for Maya

File: src/maya_description/urdf/common_properties.xacro (robot description, xacro)
@@ -1,5 +1,5 @@
 <?xml version="1.0"?>
 <robot xmlns:xacro="http://www.ros.org/wiki/xacro">
-  <!-- brief Global materials shared by Maya -->
+  <!-- Global materials shared by Maya -->
   <material name="maya_body">
     <color rgba="0.6 0.0 0.0 1.0"/>
@@ -8,46 +8,93 @@
     <color rgba="0.7 0.7 0.7 1.0"/>
   </material>
-  <!-- brief Mesh scale factor for all STL geometry -->
-  <!-- If meshes are exported in millimeters set mesh_scale to 0.001 -->
+  <!-- Mesh scale factor for all STL geometry.
+       If meshes are exported in millimeters set mesh_scale to 0.001 -->
   <xacro:property name="mesh_scale" value="1.0"/>
-  <!-- brief Vertical offset from base_footprint to base_link origin -->
-  <!-- base_footprint is on ground plane -->
+  <!-- Vertical offset from base_footprint to base_link origin.
+       base_footprint is on ground plane -->
   <xacro:property name="footprint_z" value="0.424"/>
-  <!-- brief Base link visual and collision mesh offset relative to base_link frame -->
-  <!-- This compensates CAD export so robot origin is centered for navigation -->
+  <!-- Base link visual and collision mesh offset relative to base_link frame.
+       This compensates CAD export so robot origin is centered for navigation -->
   <xacro:property name="base_link_mesh_offset_xyz" value="0.4 0 0"/>
   <xacro:property name="base_link_mesh_offset_rpy" value="0 0 0"/>
-  <!-- brief Base link inertial parameters in base_link frame -->
-  <!-- COM was exported at minus 0.39811 in X then mesh was shifted plus 0.4 -->
-  <!-- New COM X is minus 0.39811 plus 0.4 equals 0.00189 -->
-  <xacro:property name="base_inertial_xyz" value="0.00189 -0.10577 0.1455"/>
-  <xacro:property name="base_inertial_rpy" value="0 0 0"/>
+  <!-- Base link inertial parameters in base_link frame (approximate).
+       COM was exported at -0.39811 in X then mesh was shifted +0.4
+       New COM X is -0.39811 + 0.4 = 0.00189 -->
+  <xacro:property name="base_inertial_xyz" value="0.00189 -0.10577 0.1"/>
+  <xacro:property name="base_inertial_rpy" value="${half_pi} 0 0"/>
+  <!-- Total mass of the base assembly (chassis, according to your CAD) -->
   <xacro:property name="base_mass" value="24.919"/>
-  <!-- brief Base link inertia tensor components in kg m2 -->
-  <xacro:property name="base_ixx" value="4.3782"/>
-  <xacro:property name="base_ixy" value="0.048897"/>
-  <xacro:property name="base_ixz" value="0.11401"/>
-  <xacro:property name="base_iyy" value="6.5909"/>
-  <xacro:property name="base_iyz" value="0.075761"/>
-  <xacro:property name="base_izz" value="3.9583"/>
-  <!-- brief Wheel inertial properties shared by four wheels -->
+  <!-- ============================================================= -->
+  <!-- Geometric + inertial convenience properties and macros        -->
+  <!-- ============================================================= -->
+  <!-- Approximate base geometry (meters) – tune these to match the real rover.
+       length = X, width = Y, height = Z in the base_link frame -->
+  <xacro:property name="base_length" value="0.80"/>
+  <xacro:property name="base_width"  value="0.70"/>
+  <xacro:property name="base_height" value="0.30"/>
+  <!-- Wheel geometry (using drive_wheel_radius defined below) -->
+  <xacro:property name="wheel_radius" value="${drive_wheel_radius}"/>
+  <!-- Approximate wheel width (meters) – tune as needed -->
+  <xacro:property name="wheel_width" value="0.05"/>
+  <!-- Wheel mass (per wheel) – matches your existing value -->
   <xacro:property name="wheel_mass" value="1.93267"/>
-  <xacro:property name="wheel_ixx"  value="0.0080174"/>
-  <xacro:property name="wheel_iyy"  value="0.0080173"/>
-  <xacro:property name="wheel_izz"  value="0.014159"/>
-  <!-- brief Off diagonal terms taken from CAD and assumed equal for all wheels -->
-  <xacro:property name="wheel_ixy" value="1.3553E-08"/>
-  <xacro:property name="wheel_ixz" value="-2.7525E-09"/>
-  <xacro:property name="wheel_iyz" value="1.3936E-09"/>
-  <!-- brief Default wheel spin axes -->
-  <!-- Left wheels use positive Z -->
-  <!-- Right wheels use negative Z to compensate CAD mirroring -->
+  <!-- Box inertia macro for a box centered at the link frame,
+       aligned with axes. Arguments:
+       m is mass, w is width (Y), d is length (X), h is height (Z) -->
+  <xacro:macro name="box_inertia" params="m w d h xyz:='0 0 0' rpy:='0 0 0'">
+    <inertial>
+      <origin xyz="${xyz}" rpy="${rpy}"/>
+      <mass value="${m}"/>
+      <inertia
+        ixx="${(m/12.0) * (h*h + d*d)}"
+        ixy="0.0"
+        ixz="0.0"
+        iyy="${(m/12.0) * (w*w + d*d)}"
+        iyz="0.0"
+        izz="${(m/12.0) * (w*w + h*h)}"/>
+    </inertial>
+  </xacro:macro>
+  <!-- Cylinder inertia macro for a cylinder aligned with Z-axis,
+       centered at the link frame.
+       m is mass, r is radius, h is length along Z.
+       xyz / rpy let you shift/rotate the inertial origin. -->
+  <xacro:macro name="cylinder_inertia" params="m r h xyz:='0 0 0' rpy:='0 0 0'">
+    <inertial>
+      <origin xyz="${xyz}" rpy="${rpy}"/>
+      <mass value="${m}"/>
+      <inertia
+        ixx="${(m/12.0) * (3.0*r*r + h*h)}"
+        ixy="0.0"
+        ixz="0.0"
+        iyy="${(m/12.0) * (3.0*r*r + h*h)}"
+        iyz="0.0"
+        izz="${(m/2.0) * (r*r)}"/>
+    </inertial>
+  </xacro:macro>
+  <!-- Sphere inertia macro for a solid sphere centered at the link frame.
+       Currently unused, but kept for future caster wheels. -->
+  <xacro:macro name="sphere_inertia" params="m r">
+    <inertial>
+      <origin xyz="0 0 0" rpy="0 0 0"/>
+      <mass value="${m}"/>
+      <inertia
+        ixx="${(2.0/5.0) * m * (r*r)}"
+        ixy="0.0"
+        ixz="0.0"
+        iyy="${(2.0/5.0) * m * (r*r)}"
+        iyz="0.0"
+        izz="${(2.0/5.0) * m * (r*r)}"/>
+    </inertial>
+  </xacro:macro>
+  <!-- Default wheel spin axes.
+       Left wheels use positive Z, right wheels use negative Z
+       to compensate CAD mirroring. -->
   <xacro:property name="wheel_axis_left"  value="0 0 1"/>
   <xacro:property name="wheel_axis_right" value="0 0 -1"/>
-  <!-- brief Helper constant for quarter turn about Z -->
+  <!-- Helper constant for quarter turn about Z -->
   <xacro:property name="half_pi" value="${pi / 2.0}"/>
-  <!-- brief Gazebo drive parameters for skid steer model -->
-  <!-- wheel_separation is lateral distance between left and right wheel centers -->
-  <!-- wheel_radius is effective rolling radius -->
+  <!-- Gazebo drive parameters for skid steer model.
+       wheel_separation is lateral distance between left/right wheel centers.
+       drive_wheel_radius is effective rolling radius. -->
   <xacro:property name="drive_wheel_separation" value="0.785"/>
   <xacro:property name="drive_wheel_radius"      value="0.10"/>

File: src/maya_description/urdf/mobile_base.xacro (robot description, xacro)
@@ -1,12 +1,14 @@
 <?xml version="1.0"?>
 <robot xmlns:xacro="http://www.ros.org/wiki/xacro">
-  <!-- brief Base link carries inertial, visual and collision for Maya -->
+  <!-- Base link carries inertial, visual and collision for Maya -->
   <link name="base_link">
-    <inertial>
-      <origin xyz="${base_inertial_xyz}" rpy="${base_inertial_rpy}"/>
-      <mass value="${base_mass}"/>
-      <inertia ixx="${base_ixx}" ixy="${base_ixy}" ixz="${base_ixz}"
-               iyy="${base_iyy}" iyz="${base_iyz}" izz="${base_izz}"/>
-    </inertial>
+    <!-- Base inertia approximated as axis-aligned box using base dimensions -->
+    <xacro:box_inertia
+      m="${base_mass}"
+      w="${base_width}"
+      d="${base_length}"
+      h="${base_height}"
+      xyz="${base_inertial_xyz}"
+      rpy="${base_inertial_rpy}"/>
     <visual>
       <origin xyz="${base_link_mesh_offset_xyz}" rpy="${base_link_mesh_offset_rpy}"/>
@@ -25,6 +27,6 @@
     </collision>
   </link>
-  <!-- brief Ground level helper frame for navigation -->
-  <!-- base_footprint has ROS convention axes -->
+  <!-- Ground level helper frame for navigation.
+       base_footprint has ROS convention axes -->
   <link name="base_footprint"/>
   <joint name="base_joint" type="fixed">
@@ -34,5 +36,5 @@
     <origin xyz="0 0 ${footprint_z}" rpy="0 0 ${half_pi}"/>
   </joint>
-  <!-- brief Generic wheel macro with inertial, visual and continuous joint -->
+  <!-- Generic wheel macro with inertial, visual and continuous joint -->
   <xacro:macro name="maya_wheel"
                params="prefix mesh
@@ -40,10 +42,12 @@
                        inertial_xyz:='0 0 0' inertial_rpy:='0 0 0'">
     <link name="${prefix}">
-      <inertial>
-        <origin xyz="${inertial_xyz}" rpy="${inertial_rpy}"/>
-        <mass value="${wheel_mass}"/>
-        <inertia ixx="${wheel_ixx}" ixy="${wheel_ixy}" ixz="${wheel_ixz}"
-                 iyy="${wheel_iyy}" iyz="${wheel_iyz}" izz="${wheel_izz}"/>
-      </inertial>
+      <!-- Wheel inertia approximated as solid cylinder
+           COM and orientation taken from inertial_xyz / inertial_rpy -->
+      <xacro:cylinder_inertia
+        m="${wheel_mass}"
+        r="${wheel_radius}"
+        h="${wheel_width}"
+        xyz="${inertial_xyz}"
+        rpy="${inertial_rpy}"/>
       <visual>
         <origin xyz="0 0 0" rpy="0 0 0"/>
@@ -69,5 +73,5 @@
     </joint>
   </xacro:macro>
-  <!-- brief Left wheels use default spin axis from wheel_axis_left -->
+  <!-- Left wheels use default spin axis from wheel_axis_left -->
   <xacro:maya_wheel
       prefix="front_left"
@@ -84,5 +88,5 @@
       inertial_xyz="-4.8481E-06 -8.0801E-06 -0.057572"
       inertial_rpy="0 0 0"/>
-  <!-- brief Right wheels override spin axis to wheel_axis_right -->
+  <!-- Right wheels override spin axis to wheel_axis_right -->
   <xacro:maya_wheel
       prefix="front_right"

Commit message: feat(maya): slam + nav2 bringup

File: src/maya_description/urdf/common_properties.xacro (robot description, xacro)
@@ -3,8 +3,8 @@
   <!-- Global materials shared by Maya -->
   <material name="maya_body">
-    <color rgba="0.6 0.0 0.0 1.0"/>
+    <color rgba="0.0 0.38 0.45 1.0"/>
   </material>
   <material name="maya_wheel">
-    <color rgba="0.7 0.7 0.7 1.0"/>
+    <color rgba="0.05 0.05 0.05 1.0"/>
   </material>
   <!-- Mesh scale factor for all STL geometry.
@@ -13,16 +13,20 @@
   <!-- Vertical offset from base_footprint to base_link origin.
        base_footprint is on ground plane -->
-  <xacro:property name="footprint_z" value="0.424"/>
+  <xacro:property name="footprint_z" value="0.44"/>
   <!-- Base link visual and collision mesh offset relative to base_link frame.
        This compensates CAD export so robot origin is centered for navigation -->
-  <xacro:property name="base_link_mesh_offset_xyz" value="0.4 0 0"/>
+  <xacro:property name="base_link_mesh_offset_xyz" value="0.0705 -0.16 0.01"/>
   <xacro:property name="base_link_mesh_offset_rpy" value="0 0 0"/>
-  <!-- Base link inertial parameters in base_link frame (approximate).
-       COM was exported at -0.39811 in X then mesh was shifted +0.4
-       New COM X is -0.39811 + 0.4 = 0.00189 -->
-  <xacro:property name="base_inertial_xyz" value="0.00189 -0.10577 0.1"/>
-  <xacro:property name="base_inertial_rpy" value="${half_pi} 0 0"/>
+  <!-- Base link inertial parameters in base_link frame (from CAD) -->
+  <xacro:property name="base_inertial_xyz" value="0 0 0.13"/>
+  <xacro:property name="base_inertial_rpy" value="0 0 0"/>
+  <xacro:property name="base_inertia_ixx" value="0.11833"/>
+  <xacro:property name="base_inertia_ixy" value="-1.7951E-05"/>
+  <xacro:property name="base_inertia_ixz" value="-7.1707E-06"/>
+  <xacro:property name="base_inertia_iyy" value="0.20257"/>
+  <xacro:property name="base_inertia_iyz" value="-0.0006245"/>
+  <xacro:property name="base_inertia_izz" value="0.13032"/>
   <!-- Total mass of the base assembly (chassis, according to your CAD) -->
-  <xacro:property name="base_mass" value="24.919"/>
+  <xacro:property name="base_mass" value="25"/>
   <!-- ============================================================= -->
   <!-- Geometric + inertial convenience properties and macros        -->
@@ -37,6 +41,14 @@
   <!-- Approximate wheel width (meters) – tune as needed -->
   <xacro:property name="wheel_width" value="0.05"/>
-  <!-- Wheel mass (per wheel) – matches your existing value -->
-  <xacro:property name="wheel_mass" value="1.93267"/>
+  <!-- Wheel mass (per wheel) – from CAD -->
+  <xacro:property name="wheel_mass" value="1.4536"/>
+  <xacro:property name="wheel_inertial_xyz" value="1.0324E-05 1.5584E-05 -0.15844"/>
+  <xacro:property name="wheel_inertial_rpy" value="0 0 0"/>
+  <xacro:property name="wheel_inertia_ixx" value="0.014265"/>
+  <xacro:property name="wheel_inertia_ixy" value="-1.2792E-07"/>
+  <xacro:property name="wheel_inertia_ixz" value="-1.0752E-07"/>
+  <xacro:property name="wheel_inertia_iyy" value="0.014264"/>
+  <xacro:property name="wheel_inertia_iyz" value="-9.6151E-08"/>
+  <xacro:property name="wheel_inertia_izz" value="0.025537"/>
   <!-- Box inertia macro for a box centered at the link frame,
        aligned with axes. Arguments:
@@ -97,5 +109,5 @@
        wheel_separation is lateral distance between left/right wheel centers.
        drive_wheel_radius is effective rolling radius. -->
-  <xacro:property name="drive_wheel_separation" value="0.785"/>
-  <xacro:property name="drive_wheel_radius"      value="0.10"/>
+  <xacro:property name="drive_wheel_separation" value="1.09449"/>
+  <xacro:property name="drive_wheel_radius"     value="0.1636"/>
 </robot>

File: src/maya_description/urdf/mobile_base.xacro (robot description, xacro)
@@ -3,6 +3,16 @@
   <!-- Base link carries inertial, visual and collision for Maya -->
   <link name="base_link">
-    <!-- Base inertia approximated as axis-aligned box using base dimensions -->
-    <xacro:box_inertia m="${base_mass}" w="${base_width}" d="${base_length}" h="${base_height}" xyz="${base_inertial_xyz}" rpy="${base_inertial_rpy}"/>
+    <!-- Base inertia from CAD -->
+    <inertial>
+      <origin xyz="${base_inertial_xyz}" rpy="${base_inertial_rpy}"/>
+      <mass value="${base_mass}"/>
+      <inertia
+        ixx="${base_inertia_ixx}"
+        ixy="${base_inertia_ixy}"
+        ixz="${base_inertia_ixz}"
+        iyy="${base_inertia_iyy}"
+        iyz="${base_inertia_iyz}"
+        izz="${base_inertia_izz}"/>
+    </inertial>
     <visual>
       <origin xyz="${base_link_mesh_offset_xyz}" rpy="${base_link_mesh_offset_rpy}"/>
@@ -31,7 +41,16 @@
   <xacro:macro name="maya_wheel" params="prefix mesh xyz:='0 0 0' rpy:='0 0 0' axis:='${wheel_axis_left}' inertial_xyz:='0 0 0' inertial_rpy:='0 0 0'">
     <link name="${prefix}">
-      <!-- Wheel inertia approximated as solid cylinder
-           COM and orientation taken from inertial_xyz / inertial_rpy -->
-      <xacro:cylinder_inertia m="${wheel_mass}" r="${wheel_radius}" h="${wheel_width}" xyz="${inertial_xyz}" rpy="${inertial_rpy}"/>
+      <!-- Wheel inertia from CAD -->
+      <inertial>
+        <origin xyz="${wheel_inertial_xyz}" rpy="${wheel_inertial_rpy}"/>
+        <mass value="${wheel_mass}"/>
+        <inertia
+          ixx="${wheel_inertia_ixx}"
+          ixy="${wheel_inertia_ixy}"
+          ixz="${wheel_inertia_ixz}"
+          iyy="${wheel_inertia_iyy}"
+          iyz="${wheel_inertia_iyz}"
+          izz="${wheel_inertia_izz}"/>
+      </inertial>
       <visual>
         <origin xyz="0 0 0" rpy="0 0 0"/>
@@ -42,5 +61,5 @@
       </visual>
       <collision>
-        <origin xyz="0 0 0" rpy="0 0 0"/>
+          <origin xyz="0 0 0" rpy="0 0 0"/>
         <geometry>
           <mesh filename="${mesh}" scale="${mesh_scale} ${mesh_scale} ${mesh_scale}"/>
@@ -56,8 +75,8 @@
   </xacro:macro>
   <!-- Left wheels use default spin axis from wheel_axis_left -->
-  <xacro:maya_wheel prefix="front_left" mesh="file://$(find maya_description)/meshes/front_left.STL" xyz="-0.38478 -0.62736 -0.27744" rpy="1.5702 0 1.5708" inertial_xyz="-4.8481E-06 -8.0801E-06 -0.057753" inertial_rpy="0 0 0"/>
-  <xacro:maya_wheel prefix="back_left" mesh="file://$(find maya_description)/meshes/back_left.STL" xyz="-0.38513 0.28848 -0.27699" rpy="1.5708 0 1.5708" inertial_xyz="-4.8481E-06 -8.0801E-06 -0.057572" inertial_rpy="0 0 0"/>
+  <xacro:maya_wheel prefix="front_left" mesh="file://$(find maya_description)/meshes/front_left.STL" xyz="-0.32478 -0.62736 -0.27744" rpy="1.5702 0 1.5708" inertial_xyz="-4.8481E-06 -8.0801E-06 -0.057753" inertial_rpy="0 0 0"/>
+  <xacro:maya_wheel prefix="back_left" mesh="file://$(find maya_description)/meshes/back_left.STL" xyz="-0.32513 0.28848 -0.27699" rpy="1.5708 0 1.5708" inertial_xyz="-4.8481E-06 -8.0801E-06 -0.057572" inertial_rpy="0 0 0"/>
   <!-- Right wheels override spin axis to wheel_axis_right -->
-  <xacro:maya_wheel prefix="front_right" mesh="file://$(find maya_description)/meshes/front_right.STL" xyz="0.3987596 -0.61714 -0.27409" rpy="1.5657 0.51887 -1.5734" axis="${wheel_axis_right}" inertial_xyz="-4.8512E-06 -8.0627E-06 -0.046342" inertial_rpy="0 0 0"/>
-  <xacro:maya_wheel prefix="back_right" mesh="file://$(find maya_description)/meshes/back_right.STL" xyz="0.4012382 0.27364 -0.28031" rpy="-1.5781 -0.91737 1.5766" axis="${wheel_axis_right}" inertial_xyz="-4.8659E-06 -8.069E-06 -0.034709" inertial_rpy="0 0 0"/>
+  <xacro:maya_wheel prefix="front_right" mesh="file://$(find maya_description)/meshes/front_right.STL" xyz="0.3112596 -0.61714 -0.27409" rpy="1.5657 0.51887 -1.5734" axis="${wheel_axis_right}" inertial_xyz="-4.8512E-06 -8.0627E-06 -0.046342" inertial_rpy="0 0 0"/>
+  <xacro:maya_wheel prefix="back_right" mesh="file://$(find maya_description)/meshes/back_right.STL" xyz="0.3112382 0.27364 -0.28031" rpy="-1.5781 -0.91737 1.5766" axis="${wheel_axis_right}" inertial_xyz="-4.8659E-06 -8.069E-06 -0.034709" inertial_rpy="0 0 0"/>
 </robot>

File: src/maya_description/urdf/mobile_base_gazebo.xacro (robot description, xacro)
@@ -5,9 +5,9 @@
     <plugin filename="gz-sim-diff-drive-system" name="gz::sim::systems::DiffDrive">
       <!-- Left side joints for skid steer -->
-      <left_joint>front_left_joint</left_joint>
-      <left_joint>back_left_joint</left_joint>
+      <left_joint>front_right_joint</left_joint>
+      <left_joint>back_right_joint</left_joint>
       <!-- Right side joints for skid steer -->
-      <right_joint>front_right_joint</right_joint>
-      <right_joint>back_right_joint</right_joint>
+      <right_joint>front_left_joint</right_joint>
+      <right_joint>back_left_joint</right_joint>
       <!-- Frames consistent with ROS navigation stack -->
       <frame_id>odom</frame_id>

File: src/maya_description/urdf/sensors.xacro (robot description, xacro)
@@ -1,78 +1,5 @@
 <?xml version="1.0"?>
 <robot xmlns:xacro="http://www.ros.org/wiki/xacro">
-  <!-- IMU Link and Joint -->
-  <link name="imu_link">
-    <inertial>
-      <mass value="0.01"/>
-      <origin xyz="0 0 0" rpy="0 0 0"/>
-      <inertia ixx="0.00001" ixy="0" ixz="0" iyy="0.00001" iyz="0" izz="0.00001"/>
-    </inertial>
-  </link>
-  <joint name="imu_joint" type="fixed">
-    <parent link="base_link"/>
-    <child link="imu_link"/>
-    <origin xyz="0 0 0" rpy="0 0 0"/>
-  </joint>
-  <!-- LiDAR Link and Joint -->
-  <link name="lidar_link">
-    <inertial>
-      <mass value="0.1"/>
-      <origin xyz="0 0 0" rpy="0 0 0"/>
-      <inertia ixx="0.0001" ixy="0" ixz="0" iyy="0.0001" iyz="0" izz="0.0001"/>
-    </inertial>
-    <visual>
-      <geometry>
-        <cylinder radius="0.05" length="0.05"/>
-      </geometry>
-      <material name="black">
-        <color rgba="0 0 0 1"/>
-      </material>
-    </visual>
-  </link>
-  <joint name="lidar_joint" type="fixed">
-    <parent link="base_link"/>
-    <child link="lidar_link"/>
-    <origin xyz="0 0 0.3" rpy="0 0 0"/>
-  </joint>
-  <!-- IMU Sensor Plugin -->
-  <gazebo reference="imu_link">
-    <sensor name="imu_sensor" type="imu">
-      <always_on>1</always_on>
-      <update_rate>100</update_rate>
-      <visualize>true</visualize>
-      <topic>imu</topic>
-    </sensor>
-  </gazebo>
-  <!-- LiDAR Sensor Plugin -->
-  <gazebo reference="lidar_link">
-    <sensor name="lidar" type="gpu_lidar">
-      <pose>0 0 0 0 0 0</pose>
-      <always_on>true</always_on>
-      <visualize>true</visualize>
-      <update_rate>10</update_rate>
-      <topic>scan</topic>
-      <gz_frame_id>lidar_link</gz_frame_id>
-      <ray>
-        <scan>
-          <horizontal>
-            <samples>360</samples>
-            <resolution>1</resolution>
-            <min_angle>-3.14</min_angle>
-            <max_angle>3.14</max_angle>
-          </horizontal>
-          <vertical>
-            <samples>1</samples>
-            <resolution>0.01</resolution>
-            <min_angle>0</min_angle>
-            <max_angle>0</max_angle>
-          </vertical>
-        </scan>
-        <range>
-          <min>0.08</min>
-          <max>10.0</max>
-          <resolution>0.01</resolution>
-        </range>
-      </ray>
-    </sensor>
-  </gazebo>
+  <xacro:include filename="$(find maya_description)/urdf/sensors_frames.xacro"/>
+  <xacro:include filename="$(find maya_description)/urdf/sensors_gazebo.xacro"/>
 </robot>
