Commit message: Checkpoint spin diagnostics and stabilize sim odom baseline

File: src/maya_description/urdf/common_properties.xacro (robot description, xacro)
@@ -100,6 +100,6 @@
   </xacro:macro>
   <!-- Default wheel spin axes.
-       Left wheels use positive Z, right wheels use negative Z
-       to compensate CAD mirroring. -->
+       Right wheels keep the mirrored sign required by the current Maya CAD and
+       Gazebo drive setup. Normalizing the sign regressed actual body rotation. -->
   <xacro:property name="wheel_axis_left"  value="0 0 1"/>
   <xacro:property name="wheel_axis_right" value="0 0 -1"/>

File: src/maya_description/urdf/mobile_base.xacro (robot description, xacro)
@@ -61,7 +61,9 @@
       </visual>
       <collision>
-          <origin xyz="0 0 0" rpy="0 0 0"/>
+        <!-- Use a simple cylinder for wheel-ground contact in simulation.
+             Mesh collisions make skid-steer contact unstable and corrupt turning. -->
+        <origin xyz="0 0 0" rpy="0 0 0"/>
         <geometry>
-          <mesh filename="${mesh}" scale="${mesh_scale} ${mesh_scale} ${mesh_scale}"/>
+          <cylinder radius="${wheel_radius}" length="${wheel_width}"/>
         </geometry>
       </collision>

File: src/maya_description/urdf/mobile_base_gazebo.xacro (robot description, xacro)
@@ -4,10 +4,10 @@
   <gazebo>
     <plugin filename="gz-sim-diff-drive-system" name="gz::sim::systems::DiffDrive">
-      <!-- Left side joints for skid steer -->
-      <left_joint>front_right_joint</left_joint>
-      <left_joint>back_right_joint</left_joint>
-      <!-- Right side joints for skid steer -->
-      <right_joint>front_left_joint</right_joint>
-      <right_joint>back_left_joint</right_joint>
+      <!-- Match Gazebo wheel groups to the actual rover left/right sides.
+           Swapping these corrupts turn kinematics and poisons /odom yaw. -->
+      <left_joint>front_left_joint</left_joint>
+      <left_joint>back_left_joint</left_joint>
+      <right_joint>front_right_joint</right_joint>
+      <right_joint>back_right_joint</right_joint>
       <!-- Frames consistent with ROS navigation stack -->
       <frame_id>odom</frame_id>
@@ -24,4 +24,30 @@
     </plugin>
   </gazebo>
+  <!-- Give the drive wheels explicit contact parameters for skid-steer turning.
+       Heightmap terrain is much less forgiving than the empty world defaults. -->
+  <gazebo reference="front_left">
+    <mu1>1.2</mu1>
+    <mu2>1.2</mu2>
+    <slip1>0.02</slip1>
+    <slip2>0.02</slip2>
+  </gazebo>
+  <gazebo reference="back_left">
+    <mu1>1.2</mu1>
+    <mu2>1.2</mu2>
+    <slip1>0.02</slip1>
+    <slip2>0.02</slip2>
+  </gazebo>
+  <gazebo reference="front_right">
+    <mu1>1.2</mu1>
+    <mu2>1.2</mu2>
+    <slip1>0.02</slip1>
+    <slip2>0.02</slip2>
+  </gazebo>
+  <gazebo reference="back_right">
+    <mu1>1.2</mu1>
+    <mu2>1.2</mu2>
+    <slip1>0.02</slip1>
+    <slip2>0.02</slip2>
+  </gazebo>
   <gazebo>
     <plugin filename="gz-sim-imu-system" name="gz::sim::systems::Imu">

Commit message: Integrate validated minimal odom baseline

File: src/maya_description/urdf/common_properties.xacro (robot description, xacro)
@@ -109,5 +109,5 @@
        wheel_separation is lateral distance between left/right wheel centers.
        drive_wheel_radius is effective rolling radius. -->
-  <xacro:property name="drive_wheel_separation" value="1.09449"/>
+  <xacro:property name="drive_wheel_separation" value="1.0"/>
   <xacro:property name="drive_wheel_radius"     value="0.1636"/>
 </robot>

Commit message: release: promote stable gnss waypoint navigation

File: src/maya_description/urdf/common_properties.xacro (robot description, xacro)
@@ -111,5 +111,5 @@
        wheel_separation is lateral distance between left/right wheel centers.
        drive_wheel_radius is effective rolling radius. -->
-  <xacro:property name="drive_wheel_separation" value="1.09449"/>
+  <xacro:property name="drive_wheel_separation" value="1.0"/>
   <xacro:property name="drive_wheel_radius"     value="0.1636"/>
 </robot>

File: src/maya_description/urdf/mobile_base.xacro (robot description, xacro)
@@ -18,5 +18,5 @@
       <origin xyz="${base_link_mesh_offset_xyz}" rpy="${base_link_mesh_offset_rpy}"/>
       <geometry>
-        <mesh filename="file://$(find maya_description)/meshes/base_link.STL" scale="${mesh_scale} ${mesh_scale} ${mesh_scale}"/>
+        <mesh filename="package://maya_description/meshes/base_link.STL" scale="${mesh_scale} ${mesh_scale} ${mesh_scale}"/>
       </geometry>
       <material name="maya_body"/>
@@ -25,5 +25,5 @@
       <origin xyz="${base_link_mesh_offset_xyz}" rpy="${base_link_mesh_offset_rpy}"/>
       <geometry>
-        <mesh filename="file://$(find maya_description)/meshes/base_link.STL" scale="${mesh_scale} ${mesh_scale} ${mesh_scale}"/>
+        <mesh filename="package://maya_description/meshes/base_link.STL" scale="${mesh_scale} ${mesh_scale} ${mesh_scale}"/>
       </geometry>
     </collision>
@@ -61,9 +61,7 @@
       </visual>
       <collision>
-        <!-- Use a simple cylinder for wheel-ground contact in simulation.
-             Mesh collisions make skid-steer contact unstable and corrupt turning. -->
-        <origin xyz="0 0 0" rpy="0 0 0"/>
+          <origin xyz="0 0 0" rpy="0 0 0"/>
         <geometry>
-          <cylinder radius="${wheel_radius}" length="${wheel_width}"/>
+          <mesh filename="${mesh}" scale="${mesh_scale} ${mesh_scale} ${mesh_scale}"/>
         </geometry>
       </collision>
@@ -76,12 +74,9 @@
     </joint>
   </xacro:macro>
-  <!-- Wheel joint Z values are leveled for Gazebo contact. The CAD-exported
-       wheel origins differed by a few millimeters, enough to make one wheel
-       float or overload another during skid-steer turns. -->
   <!-- Left wheels use default spin axis from wheel_axis_left -->
-  <xacro:maya_wheel prefix="front_left" mesh="file://$(find maya_description)/meshes/front_left.STL" xyz="-0.32478 -0.62736 -0.2764" rpy="1.5702 0 1.5708" inertial_xyz="-4.8481E-06 -8.0801E-06 -0.057753" inertial_rpy="0 0 0"/>
-  <xacro:maya_wheel prefix="back_left" mesh="file://$(find maya_description)/meshes/back_left.STL" xyz="-0.32513 0.28848 -0.2764" rpy="1.5708 0 1.5708" inertial_xyz="-4.8481E-06 -8.0801E-06 -0.057572" inertial_rpy="0 0 0"/>
+  <xacro:maya_wheel prefix="front_left" mesh="package://maya_description/meshes/front_left.STL" xyz="-0.32478 -0.62736 -0.27744" rpy="1.5702 0 1.5708" inertial_xyz="-4.8481E-06 -8.0801E-06 -0.057753" inertial_rpy="0 0 0"/>
+  <xacro:maya_wheel prefix="back_left" mesh="package://maya_description/meshes/back_left.STL" xyz="-0.32513 0.28848 -0.27699" rpy="1.5708 0 1.5708" inertial_xyz="-4.8481E-06 -8.0801E-06 -0.057572" inertial_rpy="0 0 0"/>
   <!-- Right wheels override spin axis to wheel_axis_right -->
-  <xacro:maya_wheel prefix="front_right" mesh="file://$(find maya_description)/meshes/front_right.STL" xyz="0.3112596 -0.61714 -0.2764" rpy="1.5657 0.51887 -1.5734" axis="${wheel_axis_right}" inertial_xyz="-4.8512E-06 -8.0627E-06 -0.046342" inertial_rpy="0 0 0"/>
-  <xacro:maya_wheel prefix="back_right" mesh="file://$(find maya_description)/meshes/back_right.STL" xyz="0.3112382 0.27364 -0.2764" rpy="-1.5781 -0.91737 1.5766" axis="${wheel_axis_right}" inertial_xyz="-4.8659E-06 -8.069E-06 -0.034709" inertial_rpy="0 0 0"/>
+  <xacro:maya_wheel prefix="front_right" mesh="package://maya_description/meshes/front_right.STL" xyz="0.3112596 -0.61714 -0.27409" rpy="1.5657 0.51887 -1.5734" axis="${wheel_axis_right}" inertial_xyz="-4.8512E-06 -8.0627E-06 -0.046342" inertial_rpy="0 0 0"/>
+  <xacro:maya_wheel prefix="back_right" mesh="package://maya_description/meshes/back_right.STL" xyz="0.3112382 0.27364 -0.28031" rpy="-1.5781 -0.91737 1.5766" axis="${wheel_axis_right}" inertial_xyz="-4.8659E-06 -8.069E-06 -0.034709" inertial_rpy="0 0 0"/>
 </robot>
